Commit message: Update and rename makerspet_loki.urdf.xacro to makerspet_fido.urdf.xacro

File: urdf/makerspet_fido.urdf.xacro (robot description, xacro)
@@ -1,4 +1,4 @@
 <?xml version="1.0" ?>
-<robot name="makerspet_loki" xmlns:xacro="http://ros.org/wiki/xacro">
+<robot name="makerspet_fido" xmlns:xacro="http://ros.org/wiki/xacro">
   <!-- https://classic.gazebosim.org/tutorials?tut=ros_gzplugins&cat=connect_ros -->
   <!-- https://classic.gazebosim.org/tutorials?tut=ros_urdf&cat=connect_ros -->
@@ -281,5 +281,5 @@
       <origin xyz="0 0 0" rpy="0 0 0"/>
       <geometry>
-        <mesh filename="package://makerspet_loki/mesh/head.stl" scale="${0.001*base_diameter} ${0.001*base_diameter} ${0.001*head_height*2}"/>
+        <mesh filename="package://makerspet_fido/mesh/head.stl" scale="${0.001*base_diameter} ${0.001*base_diameter} ${0.001*head_height*2}"/>
       </geometry>
       <material name="red"/>

Commit message: URDF

File: urdf/makerspet_fido.urdf.xacro (robot description, xacro)
@@ -13,12 +13,12 @@
   <xacro:property name="caster_inset" value="0.0405"/>
   <xacro:property name="floor_clearance" value="0.018"/>
-  <xacro:property name="base_diameter" value="0.200"/>
-  <xacro:property name="wheel_base" value="0.162794"/>
-  <xacro:property name="lower_cylinder_height" value="0.119"/>
-  <xacro:property name="lower_to_upper_cylinders_gap" value="0.026"/>
-  <xacro:property name="laser_puck_to_upper_cylinder_gap" value="0.005"/>
+  <xacro:property name="base_diameter" value="0.2542"/>
+  <xacro:property name="wheel_base" value="0.214322"/>
+  <xacro:property name="lower_cylinder_height" value="0.1227"/>
+  <xacro:property name="lower_to_upper_cylinders_gap" value="0.0195"/>
+  <xacro:property name="laser_puck_to_upper_cylinder_gap" value="0.0022"/>
   <xacro:property name="laser_puck_diameter" value="0.0656"/>
-  <xacro:property name="upper_cylinder_height" value="0.013"/>
-  <xacro:property name="head_height" value="0.104"/>
+  <xacro:property name="upper_cylinder_height" value="0.003"/>
+  <xacro:property name="head_height" value="0.09"/>
   <xacro:property name="tablet_width" value="0.1669"/>
   <xacro:property name="tablet_height" value="0.0781"/>
@@ -27,5 +27,5 @@
   <xacro:property name="tablet_pitch_angle" value="20"/>
   <!-- Upper cylinder's front to tablet bottom's center -->
-  <xacro:property name="tablet_inset" value="0.055"/>
+  <xacro:property name="tablet_inset" value="0.097128"/>
   <xacro:property name="color_camera_diameter" value="0.004"/>
   <!-- Tablet edge to camera center -->

Commit message: Update makerspet_fido.urdf.xacro

File: urdf/makerspet_fido.urdf.xacro (robot description, xacro)
@@ -27,5 +27,5 @@
   <xacro:property name="tablet_pitch_angle" value="20"/>
   <!-- Upper cylinder's front to tablet bottom's center -->
-  <xacro:property name="tablet_inset" value="0.097128"/>
+  <xacro:property name="tablet_inset" value="0.07"/>
   <xacro:property name="color_camera_diameter" value="0.004"/>
   <!-- Tablet edge to camera center -->

Commit message: Update makerspet_fido.urdf.xacro

File: urdf/makerspet_fido.urdf.xacro (robot description, xacro)
@@ -11,5 +11,5 @@
   <xacro:property name="caster_diameter" value="0.042"/>
   <!-- Caster center to base edge -->
-  <xacro:property name="caster_inset" value="0.0405"/>
+  <xacro:property name="caster_inset" value="0.0386"/>
   <xacro:property name="floor_clearance" value="0.018"/>
   <xacro:property name="base_diameter" value="0.2542"/>

Commit message: Update makerspet_fido.urdf.xacro

File: urdf/makerspet_fido.urdf.xacro (robot description, xacro)
@@ -9,5 +9,5 @@
   <xacro:property name="wheel_diameter" value="0.067"/>
   <xacro:property name="wheel_width" value="0.029"/>
-  <xacro:property name="caster_diameter" value="0.042"/>
+  <xacro:property name="caster_diameter" value="0.04"/>
   <!-- Caster center to base edge -->
   <xacro:property name="caster_inset" value="0.0386"/>

Commit message: URDF sim fix

File: urdf/makerspet_fido.urdf.xacro (robot description, xacro)
@@ -189,5 +189,5 @@
     <parent link="base_link"/>
     <child link="wheel_left_link"/>
-    <origin xyz="0 ${wheel_base/2} ${wheel_diameter/2-floor_clearance}" rpy="-${pi/2} 0 0"/>
+    <origin xyz="0 ${wheel_base/2} ${wheel_diameter/2-floor_clearance}" rpy="${pi/2} 0 0"/>
     <axis xyz="0 0 1"/>
   </joint>
@@ -347,5 +347,5 @@
       <always_on>true</always_on>
       <visualize>false</visualize>
-      <update_rate>30.0</update_rate>
+      <update_rate>15.0</update_rate>
       <camera name="front_color_camera">
         <horizontal_fov>1.3962634</horizontal_fov>
@@ -415,5 +415,5 @@
     <sensor type="ray" name="laser_scan_sensor">
       <!-- pose>0 0 0 0 0 0</pose -->
-      <visualize>true</visualize>
+      <visualize>false</visualize>
       <always_on>true</always_on>
       <update_rate>9</update_rate>

Commit message: SDF cmd_vel fix

File: urdf/makerspet_fido.urdf.xacro (robot description, xacro)
@@ -39,5 +39,6 @@
   <xacro:property name="max_wheel_acceleration" value="5"/>
   <xacro:property name="lower_cylinder_mass" value="0.500"/>
-  <xacro:property name="caster_mass" value="0.020"/>
+  <!-- caster and battery weight -->
+  <xacro:property name="caster_mass" value="0.120"/>
   <xacro:property name="wheel_mass" value="0.050"/>
   <xacro:property name="laser_puck_mass" value="0.200"/>
@@ -189,5 +190,5 @@
     <parent link="base_link"/>
     <child link="wheel_left_link"/>
-    <origin xyz="0 ${wheel_base/2} ${wheel_diameter/2-floor_clearance}" rpy="${pi/2} 0 0"/>
+    <origin xyz="0 ${wheel_base/2} ${wheel_diameter/2-floor_clearance}" rpy="-${pi/2} 0 0"/>
     <axis xyz="0 0 1"/>
   </joint>
